Commit message: scaled stl files to metre units

File: src/robot_description/urdf/test.urdf (robot description, URDF)
Before this commit: robot arm, 10 links, 9 joints
Joints:
- joint joint_1: origin xyz=0 0 191.5 rpy=0 0 0 -> xyz=0 0 .1915 rpy=0 0 0
- joint joint_2: origin xyz=0 141 0 rpy=-1.57 -1.57 0 -> xyz=0 .141 0 rpy=-1.57 -1.57 0
- joint joint_3: origin xyz=230 0 -141.5 rpy=0 0 0 -> xyz=0.230 0 -0.1415 rpy=0 0 0
- joint joint_4: origin xyz=230 0 0 rpy=1.57 0 1.57 -> xyz=0.230 0 0 rpy=1.57 0 1.57
- joint joint_5: origin xyz=0 163.5 0 rpy=-1.57 0 0 -> xyz=0 0.1635 0 rpy=-1.57 0 0
- joint joint_6: origin xyz=0 -166 0 rpy=1.57 -1.57 0 -> xyz=0 -0.166 0 rpy=1.57 -1.57 0

Commit message: removed unnecessary dummy link

File: src/robot_description/urdf/test.urdf (robot description, URDF)
Before this commit: robot arm, 10 links, 9 joints
Links:
- removed link dummy_link
Joints:
- removed joint dummy_joint
- joint base_link-base: child base -> base_link; parent base_link -> base

Commit message: Scaled down Centre of mass values of links
Changed material names for gazebo reference

File: src/robot_description/urdf/test.urdf (robot description, URDF)
Before this commit: robot arm, 9 links, 8 joints
Joints:
- joint joint_1: origin xyz=0 0 .1915 rpy=0 0 0 -> xyz=0 0 0.1915 rpy=0 0 0
- joint joint_2: origin xyz=0 .141 0 rpy=-1.57 -1.57 0 -> xyz=0 0.141 0 rpy=-1.57 -1.57 0
- joint joint_4: origin xyz=0.230 0 0 rpy=1.57 0 1.57 -> xyz=0.230 0.0 0.0 rpy=1.57 0 1.57
- joint joint_5: origin xyz=0 0.1635 0 rpy=-1.57 0 0 -> xyz=0.0 0.1635 0.0 rpy=-1.57 0 0
