Commit message: Renamed some files , to be correct.
Fixed Robot to the world

File: src/robot_description/urdf/base.urdf (robot description, URDF)
Before this commit: robot arm, 9 links, 8 joints
Joints:
- joint joint_1: limit lower=-3.14 upper=3.14 effort=0 velocity=2.61 -> lower=-3.14 upper=3.14 effort=30 velocity=2.617
- joint joint_2: limit lower=-2.61 upper=2.61 effort=0 velocity=2.61 -> lower=-2.61 upper=2.61 effort=30 velocity=2.61
- joint joint_3: limit lower=-2.61 upper=2.61 effort=0 velocity=3.141 -> lower=-2.61 upper=2.61 effort=30 velocity=3.141
- joint joint_4: limit lower=-3.14 upper=3.14 effort=0 velocity=3.141 -> lower=-3.14 upper=3.14 effort=30 velocity=3.141
- joint joint_5: limit lower=-3.14 upper=3.14 effort=0 velocity=3.141 -> lower=-3.14 upper=3.14 effort=30 velocity=3.141
- joint joint_6: limit lower=-3.14 upper=3.14 effort=0 velocity=3.141 -> lower=-3.14 upper=3.14 effort=30 velocity=3.141
