Commit message: Integrated Gripper with moveit config
Added gripper to a3c description
Added gripper to a3c moveit confi
Remade pick and place cycle with new gripper orientations

File: src/a3c_description/xacro/base_mounting.xacro (robot description, xacro)
@@ -1,5 +1,5 @@
 <?xml version="1.0"?>
 <robot name="A3C" xmlns:xacro="http://wiki.ros.org/xacro">
-    <xacro:include filename="$(find a3c_moveit_config)/config/gazebo_A3C.urdf"/>
+    <xacro:include filename="$(find a3c_description)/urdf/base.urdf"/>
 	<link name="world">
 	</link>

File: src/a3c_moveit_config/config/gazebo_A3C.urdf (robot description, URDF)
Before this commit: robot A3C, 9 links, 8 joints
Links:
- added link left_inner_finger, mass 0.0104003125914103; collision mesh filename=package://a3c_description/meshes/collision/robotiq_arg2f_14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; visual mesh filename=package://a3c_description/meshes/visual/robotiq_arg2f_140_i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
- added link left_inner_finger_pad, mass 0.1; collision box size=0.03 0.07 0.0075; visual box size=0.027 0.065 0.0075
- added link left_inner_knuckle, mass 0.0271177346495152; collision mesh filename=package://a3c_description/meshes/collision/robotiq_arg2f_14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; visual mesh filename=package://a3c_description/meshes/visual/robotiq_arg2f_140_i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
- added link left_outer_finger, mass 0.022614240507152; collision mesh filename=package://a3c_description/meshes/collision/robotiq_arg2f_14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; visual mesh filename=package://a3c_description/meshes/visual/robotiq_arg2f_140_o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
- added link left_outer_knuckle, mass 0.00853198276973456; collision mesh filename=package://a3c_description/meshes/collision/robotiq_arg2f_14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; visual mesh filename=package://a3c_description/meshes/visual/robotiq_arg2f_140_o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
- added link right_inner_finger, mass 0.0104003125914103; collision mesh filename=package://a3c_description/meshes/collision/robotiq_arg2f_14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; visual mesh filename=package://a3c_description/meshes/visual/robotiq_arg2f_140_i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
- added link right_inner_finger_pad, mass 0.1; collision box size=0.03 0.07 0.0075; visual box size=0.027 0.065 0.0075
- added link right_inner_knuckle, mass 0.0271177346495152; collision mesh filename=package://a3c_description/meshes/collision/robotiq_arg2f_14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; visual mesh filename=package://a3c_description/meshes/visual/robotiq_arg2f_140_i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
- added link right_outer_finger, mass 0.022614240507152; collision mesh filename=package://a3c_description/meshes/collision/robotiq_arg2f_14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; visual mesh filename=package://a3c_description/meshes/visual/robotiq_arg2f_140_o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
- added link right_outer_knuckle, mass 0.00853198276973456; collision mesh filename=package://a3c_description/meshes/collision/robotiq_arg2f_14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; visual mesh filename=package://a3c_description/meshes/visual/robotiq_arg2f_140_o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
- added link robotiq_arg2f_base_link, mass 0.22652; collision mesh filename=package://a3c_description/meshes/collision/robotiq_arg2f_ba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; visual mesh filename=package://a3c_description/meshes/visual/robotiq_arg2f_base_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
Joints:
- added joint finger_joint: type revolute, parent robotiq_arg2f_base_link, child left_outer_knuckle, origin xyz=0 -0.030601 0.054905 rpy=2.2957963267948966 0 0, axis -1 0 0, limit lower=0 upper=0.7 effort=1000 velocity=2.0
- added joint gripper_fixture: type fixed, parent tool0, child robotiq_arg2f_base_link
- added joint left_inner_finger_joint: type revolute, parent left_outer_finger, child left_inner_finger, origin xyz=0 0.0817554015893473 -0.0282203446692936 rpy=-0.725 0 0, axis 1 0 0, limit lower=-0.8757 upper=0.8757 effort=1000 velocity=2.0, mimic joint=finger_joint multiplier=1 offset=0
- added joint left_inner_finger_pad_joint: type fixed, parent left_inner_finger, child left_inner_finger_pad, origin xyz=0 0.0457554015893473 -0.0272203446692936 rpy=0 0 0, axis 0 0 1
- added joint left_inner_knuckle_joint: type revolute, parent robotiq_arg2f_base_link, child left_inner_knuckle, origin xyz=0 -0.0127 0.06142 rpy=2.2957963267948966 0 0.0, axis 1 0 0, limit lower=-0.8757 upper=0.8757 effort=1000 velocity=2.0, mimic joint=finger_joint multiplier=-1 offset=0
- added joint left_outer_finger_joint: type fixed, parent left_outer_knuckle, child left_outer_finger, origin xyz=0 0.01821998610742 0.0260018192872234 rpy=0 0 0, axis 1 0 0
- added joint right_inner_finger_joint: type revolute, parent right_outer_finger, child right_inner_finger, origin xyz=0 0.0817554015893473 -0.0282203446692936 rpy=-0.725 0 0, axis 1 0 0, limit lower=-0.8757 upper=0.8757 effort=1000 velocity=2.0, mimic joint=finger_joint multiplier=1 offset=0
- added joint right_inner_finger_pad_joint: type fixed, parent right_inner_finger, child right_inner_finger_pad, origin xyz=0 0.0457554015893473 -0.0272203446692936 rpy=0 0 0, axis 0 0 1
- added joint right_inner_knuckle_joint: type revolute, parent robotiq_arg2f_base_link, child right_inner_knuckle, origin xyz=0 0.0127 0.06142 rpy=2.2957963267948966 0 -3.141592653589793, axis 1 0 0, limit lower=-0.8757 upper=0.8757 effort=1000 velocity=2.0, mimic joint=finger_joint multiplier=-1 offset=0
- added joint right_outer_finger_joint: type fixed, parent right_outer_knuckle, child right_outer_finger, origin xyz=0 0.01821998610742 0.0260018192872234 rpy=0 0 0, axis 1 0 0
- added joint right_outer_knuckle_joint: type revolute, parent robotiq_arg2f_base_link, child right_outer_knuckle, origin xyz=0 0.030601 0.054905 rpy=2.2957963267948966 0 3.141592653589793, axis 1 0 0, limit lower=-0.725 upper=0.725 effort=1000 velocity=2.0, mimic joint=finger_joint multiplier=-1 offset=0
