Commit message: Added Transmission for Gripper
Added mimic joints for gripper

File: src/a3c_description/xacro/robotiq_arg2f_transmission.xacro (robot description, xacro)
@@ -5,5 +5,5 @@
       <type>transmission_interface/SimpleTransmission</type>
       <joint name="${prefix}finger_joint">
-        <hardwareInterface>PositionJointInterface</hardwareInterface>
+        <hardwareInterface>hardware_interface/PositionJointInterface</hardwareInterface>
       </joint>
       <actuator name="${prefix}finger_joint_motor">
@@ -11,4 +11,33 @@
       </actuator>
     </transmission>
+    <gazebo>
+            <!-- loading plugin: mimic joints works in gazebo now-->
+            <plugin filename="libroboticsgroup_gazebo_mimic_joint_plugin.so" name="${prefix}mimic_robotiq_140_4">
+              <joint>${prefix}finger_joint</joint>
+              <mimicJoint>${prefix}right_outer_knuckle_joint</mimicJoint>
+              <multiplier>-1.0</multiplier>
+          </plugin>
+          <plugin filename="libroboticsgroup_gazebo_mimic_joint_plugin.so" name="${prefix}mimic_robotiq_140_2">
+              <joint>${prefix}finger_joint</joint>
+              <mimicJoint>${prefix}left_inner_finger_joint</mimicJoint>
+              <multiplier>1.0</multiplier>
+              <!--<offset>0.0</offset>-->
+          </plugin>
+          <plugin filename="libroboticsgroup_gazebo_mimic_joint_plugin.so" name="${prefix}mimic_robotiq_140_1">
+              <joint>${prefix}finger_joint</joint>
+              <mimicJoint>${prefix}right_inner_finger_joint</mimicJoint>
+              <multiplier>1.0</multiplier>
+          </plugin>
+          <plugin filename="libroboticsgroup_gazebo_mimic_joint_plugin.so" name="${prefix}mimic_robotiq_140_3">
+              <joint>${prefix}finger_joint</joint>
+              <mimicJoint>${prefix}left_inner_knuckle_joint</mimicJoint>
+              <multiplier>-1.0</multiplier>
+          </plugin>
+          <plugin filename="libroboticsgroup_gazebo_mimic_joint_plugin.so" name="${prefix}mimic_robotiq_140_5">
+              <joint>${prefix}finger_joint</joint>
+              <mimicJoint>${prefix}right_inner_knuckle_joint</mimicJoint>
+              <multiplier>-1.0</multiplier>
+          </plugin>
+      </gazebo>
   </xacro:macro>
 </robot>
