Commit message: Added launch files, added surface friction
Added launch files and nodes for gazebo and rviz pick_place
Added surface friction to inner pads of gripper
Added friction to outer surface of robot

File: src/a3c_description/xacro/robotiq_arg2f_140_model_macro.xacro (robot description, xacro)
@@ -144,4 +144,9 @@
       </collision>
     </link>
+    <gazebo reference="${prefix}${fingerprefix}_inner_finger_pad">
+      <material>Gazebo/Grey</material>
+      <mu1>0.2</mu1>
+      <mu2>0.2</mu2>
+    </gazebo>
   </xacro:macro>
   <xacro:macro name="outer_finger_joint" params="prefix fingerprefix">

Commit message: Correct Moveit Config
Added friction parameters in MoveIt Config

File: src/a3c_description/xacro/robotiq_arg2f_140_model_macro.xacro (robot description, xacro)
@@ -145,5 +145,4 @@
     </link>
     <gazebo reference="${prefix}${fingerprefix}_inner_finger_pad">
-      <material>Gazebo/Grey</material>
       <mu1>0.2</mu1>
       <mu2>0.2</mu2>
