Commit message: Added a minimal pick and place
Integration of grasp-fix plugin failed
has to be retired later
gazebo grasp has been implemented with a
dummy vacuumm gripper using vaccuum gripper plugin
Every a3c_moveit_config file with _vac attached, is made for running
gazebo pick and place demo with a vaccuum gripper
Effort controllers have been tuned
Added a script to remove dangling gaz and ros processes
todo:Add readmes everywhere and develop firther on robotiq gripper
grasp action later.

File: src/a3c_description/xacro/ros_control_vac.xacro (robot description, xacro)
@@ -1,5 +1,5 @@
 <?xml version="1.0"?>
 <robot name="A3C" xmlns:xacro="http://wiki.ros.org/xacro">
-    <xacro:include filename="$(find a3c_description)/xacro/gripper_mounting.xacro" />
+    <xacro:include filename="$(find a3c_description)/xacro/gripper_mounting_vac.xacro" />
 	<gazebo>
 		<plugin name="gazebo_ros_control" filename="libgazebo_ros_control.so">
@@ -63,3 +63,36 @@
 		</actuator>
 	</transmission>
+  <link name="gripper_link">
+    <gravity>0</gravity>
+    <visual>
+      <origin rpy="0 0 0" xyz="0 0 0"/>
+      <geometry>
+        <box size="0.01 0.01 0.01"/>
+      </geometry>
+      <material name="transparent">
+        <color rgba="0 0 0 0"/>
+      </material>
+    </visual>
+    <inertial>
+      <origin rpy="0 0 0" xyz="0.000000 0.000000 0.000000"/>
+      <mass value="0.0001"/>
+      <inertia ixx="1e-08" ixy="0" ixz="0" iyy="1e-08" iyz="0" izz="1e-08"/>
+    </inertial>
+  </link>
+  <joint name="gripper_joint" type="revolute">
+    <parent link="link_6" />
+    <child link="gripper_link" />
+    <origin rpy="0 0 0" xyz="0.02 0 0" />
+    <limit effort="30" velocity="1.0" lower="0" upper="0" />
+  </joint>
+  <gazebo>
+    <plugin name="gazebo_ros_vacuum_gripper" filename="libgazebo_ros_vacuum_gripper.so">
+      <robotNamespace>/A3C/</robotNamespace>
+      <bodyName>gripper_link</bodyName>
+      <topicName>grasping</topicName>
+      <maxForce>5</maxForce>
+      <maxDistance>0.10</maxDistance>
+      <minDistance>0.10</minDistance>
+    </plugin>
+  </gazebo>
 </robot>

File: src/a3c_moveit/pick_and_place/urdf/box.urdf (robot description, URDF)
Before this commit: robot simple_box, 1 links, 0 joints
Links:
- link my_box: geometry collision box size=0.05 0.05 0.02; visual box size=0.05 0.05 0.02
