Commit message: Started Moveit pick place implementation
Added a3c_moveit package
renamed robot_description to a3c_description

File: src/a3c_description/urdf/base.urdf (robot description, URDF)
Before this commit: robot A3C, 9 links, 8 joints
Links:
- link base_link: geometry collision mesh filename=package://a3c_description/meshes/l0.stl; visual mesh filename=package://a3c_description/meshes/l0.stl
- link link_1: geometry collision mesh filename=package://a3c_description/meshes/l1.stl; visual mesh filename=package://a3c_description/meshes/l1.stl
- link link_2: geometry collision mesh filename=package://a3c_description/meshes/l2.stl; visual mesh filename=package://a3c_description/meshes/l2.stl
- link link_3: geometry collision mesh filename=package://a3c_description/meshes/l3.stl; visual mesh filename=package://a3c_description/meshes/l3.stl
- link link_4: geometry collision mesh filename=package://a3c_description/meshes/l4.stl; visual mesh filename=package://a3c_description/meshes/l4.stl
- link link_5: geometry collision mesh filename=package://a3c_description/meshes/l5.stl; visual mesh filename=package://a3c_description/meshes/l5.stl
- link link_6: geometry collision mesh filename=package://a3c_description/meshes/l6.stl; visual mesh filename=package://a3c_description/meshes/l6.stl

File: src/a3c_moveit_config/config/gazebo_A3C.urdf (robot description, URDF)
Before this commit: robot A3C, 9 links, 8 joints
Links:
- link base_link: geometry collision mesh filename=package://a3c_description/meshes/l0.stl; visual mesh filename=package://a3c_description/meshes/l0.stl
- link link_1: geometry collision mesh filename=package://a3c_description/meshes/l1.stl; visual mesh filename=package://a3c_description/meshes/l1.stl
- link link_2: geometry collision mesh filename=package://a3c_description/meshes/l2.stl; visual mesh filename=package://a3c_description/meshes/l2.stl
- link link_3: geometry collision mesh filename=package://a3c_description/meshes/l3.stl; visual mesh filename=package://a3c_description/meshes/l3.stl
- link link_4: geometry collision mesh filename=package://a3c_description/meshes/l4.stl; visual mesh filename=package://a3c_description/meshes/l4.stl
- link link_5: geometry collision mesh filename=package://a3c_description/meshes/l5.stl; visual mesh filename=package://a3c_description/meshes/l5.stl
- link link_6: geometry collision mesh filename=package://a3c_description/meshes/l6.stl; visual mesh filename=package://a3c_description/meshes/l6.stl

Commit message: Realxed bounds of trajGen to get a working grasp trajectory
Added gains
Tested vaccuujm grasp successfully

File: src/a3c_description/urdf/base.urdf (robot description, URDF)
Before this commit: robot A3C, 9 links, 8 joints
Joints:
- joint joint_1: limit lower=-3.14 upper=3.14 effort=30 velocity=2.617 -> lower=-3.14 upper=3.14 effort=200 velocity=2.617
- joint joint_2: limit lower=-2.61 upper=2.61 effort=30 velocity=2.61 -> lower=-2.61 upper=2.61 effort=200 velocity=2.61
- joint joint_3: limit lower=-2.61 upper=2.61 effort=30 velocity=3.141 -> lower=-2.61 upper=2.61 effort=200 velocity=3.141
- joint joint_4: limit lower=-3.14 upper=3.14 effort=30 velocity=3.141 -> lower=-3.14 upper=3.14 effort=200 velocity=3.141
- joint joint_5: limit lower=-3.14 upper=3.14 effort=30 velocity=3.141 -> lower=-3.14 upper=3.14 effort=200 velocity=3.141
- joint joint_6: limit lower=-3.14 upper=3.14 effort=30 velocity=3.141 -> lower=-3.14 upper=3.14 effort=200 velocity=3.141

File: src/a3c_description/xacro/robotiq_arg2f_140_model_macro.xacro (robot description, xacro)
@@ -121,4 +121,8 @@
       </collision>
     </link>
+    <gazebo reference="${prefix}${fingerprefix}_inner_finger">
+        <mu1>20</mu1>
+        <mu2>20</mu2>
+    </gazebo>
   </xacro:macro>
   <!-- Finger pad link, the default are the "big pads" with rubber-->
@@ -144,8 +148,4 @@
       </collision>
     </link>
-    <gazebo reference="${prefix}${fingerprefix}_inner_finger_pad">
-      <mu1>0.2</mu1>
-      <mu2>0.2</mu2>
-    </gazebo>
   </xacro:macro>
   <xacro:macro name="outer_finger_joint" params="prefix fingerprefix">

File: src/a3c_description/xacro/robotiq_arg2f_transmission.xacro (robot description, xacro)
@@ -5,5 +5,5 @@
       <type>transmission_interface/SimpleTransmission</type>
       <joint name="${prefix}finger_joint">
-        <hardwareInterface>hardware_interface/PositionJointInterface</hardwareInterface>
+        <hardwareInterface>hardware_interface/EffortJointInterface</hardwareInterface>
       </joint>
       <actuator name="${prefix}finger_joint_motor">

File: src/a3c_description/xacro/ros_control.xacro (robot description, xacro)
@@ -63,3 +63,77 @@
 		</actuator>
 	</transmission>
+	<!-- <gazebo>
+		<plugin name="gazebo_grasp_fix" filename="libgazebo_grasp_fix.so">
+            <arm>
+                <arm_name>A3C</arm_name>
+                <palm_link>link_6</palm_link>
+                <gripper_link>left_inner_finger</gripper_link>
+                <gripper_link>right_inner_finger</gripper_link>
+            </arm>
+			<forces_angle_tolerance>91</forces_angle_tolerance>
+			<update_rate>1</update_rate>
+			<grip_count_threshold>1</grip_count_threshold>
+			<max_grip_count>10</max_grip_count>
+			<release_tolerance>0.001</release_tolerance>
+			<disable_collisions_on_attach>true</disable_collisions_on_attach>
+			<contact_topic>__default_topic__</contact_topic>
+		</plugin>
+	</gazebo> -->
+  <!-- <link name="gripper_link">
+    <gravity>0</gravity>
+    <visual>
+      <origin rpy="0 0 0" xyz="0 0 0"/>
+      <geometry>
+        <box size="0.01 0.01 0.01"/>
+      </geometry>
+      <material name="blue">
+        <color rgba="0 0 0 0"/>
+      </material>
+    </visual>
+    <inertial>
+      <origin rpy="0 0 0" xyz="0.000000 0.000000 0.000000"/>
+      <mass value="0.0001"/>
+      <inertia ixx="1e-08" ixy="0" ixz="0" iyy="1e-08" iyz="0" izz="1e-08"/>
+    </inertial>
+  </link>
+  <joint name="gripper_joint" type="revolute">
+    <parent link="link_6" />
+    <child link="gripper_link" />
+    <origin rpy="0 0 0" xyz="0.00 0 0" />
+    <limit effort="30" velocity="1.0" lower="0" upper="0" />
+  </joint>
+  <gazebo> -->
+  <link name="gripper_link">
+    <gravity>0</gravity>
+    <visual>
+      <origin rpy="0 0 0" xyz="0 0 0"/>
+      <geometry>
+        <box size="0.01 0.01 0.01"/>
+      </geometry>
+      <material name="blue">
+        <color rgba="0 0 0 0"/>
+      </material>
+    </visual>
+    <inertial>
+      <origin rpy="0 0 0" xyz="0.000000 0.000000 0.000000"/>
+      <mass value="0.0001"/>
+      <inertia ixx="1e-08" ixy="0" ixz="0" iyy="1e-08" iyz="0" izz="1e-08"/>
+    </inertial>
+  </link>
+  <joint name="gripper_joint" type="revolute">
+    <parent link="right_inner_finger" />
+    <child link="gripper_link" />
+    <origin rpy="0 0 0" xyz="0.00 0 0" />
+    <limit effort="30" velocity="1.0" lower="0" upper="0" />
+  </joint>
+  <gazebo>
+    <plugin name="gazebo_ros_vacuum_gripper" filename="libgazebo_ros_vacuum_gripper.so">
+      <robotNamespace>/A3C</robotNamespace>
+      <bodyName>gripper_link</bodyName>
+      <topicName>grasping</topicName>
+      <maxForce>50</maxForce>
+      <maxDistance>0.10</maxDistance>
+      <minDistance>0.10</minDistance>
+    </plugin>
+  </gazebo>
 </robot>

File: src/a3c_moveit/pick_and_place/urdf/box.urdf (robot description, URDF)
Before this commit: robot simple_box, 1 links, 0 joints
Links:
- link my_box: mass 1.0 -> 0.00001
